File: hw/design/jiffy.kicad_pcb (KiCad board)
At the start: 4 copper layers, 110 x 46 mm, 199 parts, among them J1 DX4R005JJ2R1800, J2 RJE72-188-1401, J3 TFM-110-02-S-D-WT, J4 Conn_01x30, J5 Conn_01x30, M1 MHNP_2.5mm, M2 MHNP_2.5mm, M3 MHNP_2.5mm, M4 MHNP_2.5mm, Q1 CSD17313Q2Q1, T1 PT61018PEL, U1 MCIMX6G2AVM07, U10 SN74AHC1G08, U11 LAN8710, U12 USBLC6-4, U13 FAN53541, U14 NCV551SN33T1G, U2 MT41K512M16HA-125, U3 LP3470M5-3.08, U4 FAN53541, U5 FAN5355UC00, U6 FEMC004GTTE7-T13-17, U7 USBLC6-4, U8 NCP360SNAET1G, U9 LM74610, X1 NX2012SA-32.768K-STD-MUB-1, X2 NX2520SA-24.000000MHZ

Commit message: R1 Release
Parts:
- J1: footprint USB_Micro-B -> Jonas:USB_Micro-B
